Commit message: Lidar height as an argument for spawning

File: multi_turtlebot_sim/urdf/turtlebot3_waffle.urdf.xacro (robot description, xacro)
@@ -8,4 +8,6 @@
     <xacro:property name="frame_prefix" value="$(arg frame_prefix)/"/>
   </xacro:if>
+  <xacro:arg name="lidar_height_arg" default="0.122"/>
+  <xacro:property name="lidar_height" value="$(arg lidar_height_arg)" />
   <xacro:arg name="topic_prefix" default=""/>
   <xacro:property name="topic_prefix" value="$(arg topic_prefix)"/>
@@ -176,5 +178,6 @@
     <parent link="base_link"/>
     <child link="base_scan"/>
-    <origin xyz="-0.064 0 0.122" rpy="0 0 0"/>
+    <origin xyz="-0.064 0 ${lidar_height}" rpy="0 0 0"/>
+     <!-- <origin xyz="-0.064 0 0.122" rpy="0 0 0"/> -->
   </joint>
   <link name="base_scan">
